File: pcb/asbmasap/asbmasap.kicad_sch (KiCad schematic)
At the start: 51 parts, among them J1 USB_C_Receptacle_USB2.0, Q1 Q_PMOS_DGS, SW1 SW_Push, U1 MCP73831-2-OT, U2 TPS61200DRC, U3 nRF52840, Y1 32.768kHz, Y2 32MHz

Commit message: feat(pcb): turn global labels into power symbols and add LCSC part number for some components
Parts:
- removed C15, C16, C19: 4.7uF, symbol Device:C_Small
- removed C6, C7, C9: 12pF, symbol Device:C
- removed R3: 5.1K, symbol Device:R
- removed Y2: 32MHz, symbol Device:Crystal
- added C? (x3): 12pF, symbol Device:C
- added C? (x2): 4.7uF, symbol Device:C_Small
- added R?: 5.1K, Resistor_SMD:R_0402_1005Metric, symbol Device:R
- added Y?: 32MHz, symbol Device:Crystal_GND24_Small
- AE1: LCSC Part (none) -> C427423; LCSC Part (alternative) (none) -> C239243
- C1, C12: LCSC Part (none) -> C368809
- C10, C13, C14, C22: LCSC Part (none) -> C1525
- C11, C17, C4: LCSC Part (none) -> C52923
- C18: LSCS Part (none) -> C307434
- C20: LCSC Part (none) -> C14442
- C21: LCSC Part (none) -> C26409
- C24: LCSC Part (none) -> C170150
- C25: LCSC Part (none) -> C371977
- C26: value 0.8pF -> 1pF; LCSC Part (none) -> C371977
- C8: LCSC Part (none) -> C184800
- J1: LCSC Part (none) -> C168688
- L2: LCSC Part (none) -> C76732
- L3: LCSC Part (none) -> C76763
- L4: LCSC Part (none) -> C354638
- R2: footprint (none) -> Resistor_SMD:R_0402_1005Metric; LCSC Part (none) -> C105872
- R5: LCSC Part (none) -> C186405
- U2: LCSC Part (none) -> C140320
- U3: LCSC Part (none) -> C1851953
- Y1: LCSC Part (none) -> C97607
Connections:
- net VDDH is gone; now on net +5V: U3.Y2 (VDDH)
- net VDD_nRF is gone; now on net +5V: C10.1, C11.1, C12.2, C13.2, C14.2, L5.1, U3.A22 (VDD), U3.AD14 (VDD), U3.AD23 (VDD), U3.B1 (VDD), U3.W1 (VDD)
- net GND: now also C?.1, C?.1, C?.2, C?.2, C?.2, R?.1, Y?.2, Y?.4
- net VBUS: now also C?.2
- net at J1.B5 (CC2): now also R?.2
- net at U3.A23 (XC2): now also C?.2, Y?.3
- net at C8.2, U3.B24 (XC1): now also Y?.1
- net at U3.D2 (XL1/P0.00), Y1.2: now also C?.1
- net at U3.F2 (XL2/P0.01), Y1.1: now also C?.1
- net 5v_OUT renamed +5V
- net DECUSB: no longer names the net of U3.AC5 (DECUSB)
- net DECUSB: now also C?.1
- no-connect marks 52 -> 54
Other:
- moved on the sheet: C10, C11, C12, C13, C14, C17, C18, C20, C21, C22, L2, L3
